Commit message: Fertiges Gazebo und Display

File: install/brokk/share/brokk/urdf/brokk170_control.xacro (robot description, xacro)
@@ -9,5 +9,5 @@
             <wheel_diameter>0.36</wheel_diameter>
             <!-- Limits -->
-            <max_wheel_torque>20000</max_wheel_torque>
+            <max_wheel_torque>200</max_wheel_torque>
             <max_wheel_acceleration>10.0</max_wheel_acceleration>
             <!-- Output -->
@@ -16,5 +16,5 @@
             <publish_odom>true</publish_odom>
             <publish_odom_tf>true</publish_odom_tf>
-            <publish_wheel_tf>true</publish_wheel_tf>
+            <publish_wheel_tf>true</publish_wheel_tf>^
         </plugin>
         <plugin name="gazebo_ros_joint_state_publisher" filename="libgazebo_ros_joint_state_publisher.so">

File: install/brokk/share/brokk/urdf/brokkmodel.xacro (robot description, xacro)
@@ -114,5 +114,5 @@
         <origin xyz="0 0 0.0" rpy="0 0 0" />
         <mass value="49.9514206426285"/>
-        <inertia ixx="0.265896" iyy="0.391346" izz="0.265896" ixy="0.0" iyz="0.0" ixz="0.0"/>>
+        <inertia ixx="0.265896" iyy="0.391346" izz="0.265896" ixy="0.0" iyz="0.0" ixz="0.0"/>
       </inertial>
   </link>
@@ -232,5 +232,5 @@
   <link name="wheel_right_behind_link">
     <visual>
-      <origin xyz="0 0 0" rpy="-0 0 0"/>
+      <origin xyz="0 0 0" rpy="0 0 0"/>
       <geometry>
         <mesh filename="file://$(find brokk)/models/meshes/wheel.stl"/>
@@ -239,5 +239,5 @@
     </visual>
     <collision>
-      <origin xyz="0 0 0.0" rpy="-0 0 0"/>
+      <origin xyz="0 0 0.0" rpy="0 0 0"/>
       <geometry>
       	<mesh filename="file://$(find brokk)/models/meshes/wheel.stl"/>
@@ -266,12 +266,12 @@
   <link name="wheel_right_mittelhinten_link">
     <visual>
-      <origin xyz="0.0 0 0.0" rpy="-0 0 0"/>
-      <geometry>
-      	<mesh filename="file://$(find brokk)/models/meshes/wheel.stl"/>
-      </geometry>
-      <material name="dark"/>
-    </visual>
-    <collision>
-      <origin xyz="0.0 0 0.0" rpy="-0 0 0"/>
+      <origin xyz="0.0 0 0.0" rpy="0 0 0"/>
+      <geometry>
+      	<mesh filename="file://$(find brokk)/models/meshes/wheel.stl"/>
+      </geometry>
+      <material name="dark"/>
+    </visual>
+    <collision>
+      <origin xyz="0.0 0 0.0" rpy="0 0 0"/>
       <geometry>
       	<mesh filename="file://$(find brokk)/models/meshes/wheel.stl"/>
@@ -301,12 +301,12 @@
   <link name="wheel_right_mittelvorne_link">
     <visual>
-      <origin xyz="0 0 0.0" rpy="-0 0 0"/>
-      <geometry>
-      	<mesh filename="file://$(find brokk)/models/meshes/wheel.stl"/>
-      </geometry>
-      <material name="dark"/>
-    </visual>
-    <collision>
-      <origin xyz="0 0 0" rpy="-0 0 0"/>
+      <origin xyz="0 0 0.0" rpy="0 0 0"/>
+      <geometry>
+      	<mesh filename="file://$(find brokk)/models/meshes/wheel.stl"/>
+      </geometry>
+      <material name="dark"/>
+    </visual>
+    <collision>
+      <origin xyz="0 0 0" rpy="0 0 0"/>
       <geometry>
       	<mesh filename="file://$(find brokk)/models/meshes/wheel.stl"/>
@@ -344,12 +344,12 @@
   <link name="wheel_right_link">
     <visual>
-      <origin xyz="0 0 0.0" rpy="-0 0 0"/>
-      <geometry>
-      	<mesh filename="file://$(find brokk)/models/meshes/wheel.stl"/>
-      </geometry>
-      <material name="dark"/>
-    </visual>
-    <collision>
-      <origin xyz="0 0 0.0" rpy="-0 0 0"/>
+      <origin xyz="0 0 0.0" rpy="0 0 0"/>
+      <geometry>
+      	<mesh filename="file://$(find brokk)/models/meshes/wheel.stl"/>
+      </geometry>
+      <material name="dark"/>
+    </visual>
+    <collision>
+      <origin xyz="0 0 0.0" rpy="0 0 0"/>
       <geometry>
       	<mesh filename="file://$(find brokk)/models/meshes/wheel.stl"/>
